Commit message: update

File: source/isaaclab_assets/isaaclab_assets/robots/uuv/hero_agent/meshes/agent.urdf (robot description, URDF)
Before this commit: robot agent, 5 links, 4 joints
Links:
- link link3: geometry collision cylinder length=0.118 radius=0.085; visual cylinder length=0.118 radius=0.085
