Commit message: feat: FullDOF-TRPO play/train support + continuous joints
- agent.urdf: joint1/joint2 revolute -> continuous (no position limits,
  cable wrapping handled by soft constraint joint1_position_cost)
- train.py: register FullDOFConstraintEncoderRunner in runner lookup
- play.py: add FullDOF-TRPO compatibility (play_mode, flexible att_err
  detection, adaptive snapshot printing for lin_vel/thruster metrics)

Co-Authored-By: Claude Opus 4.6 (1M context) <noreply@anthropic.com>

File: source/isaaclab_assets/isaaclab_assets/robots/uuv/hero_agent/meshes/agent.urdf (robot description, URDF)
Before this commit: robot agent, 5 links, 4 joints
Joints:
- joint joint1: limit lower=-6.2831853 upper=6.2831853 effort=200 velocity=30 -> effort=200 velocity=30; type revolute -> continuous
- joint joint2: limit lower=-6.2831853 upper=6.2831853 effort=200 velocity=30 -> effort=200 velocity=30; type revolute -> continuous
